File: rev/aggressor.sch (KiCad schematic (older format))
At the start: 102 parts, among them CON3_VF_MOD CONN_5, CON4_ISP CONN_6, CON5 CONN_5, IC2 MC34064P, IC3 ATMEGA32-A, SW1 DUAL_SWITCH_INV, U1 MIC5205-5.0BM5, X1 CRYSTAL

Commit message: Update schematics - newer symbols from kicad library - add external eeprom - minor visual improvements
Parts:
- removed ALT, CH1, CH2, D/R: CONN_3, symbol CONN_3
- removed ANTENNA_CON: CONN_1, symbol CONN_1
- removed BATT, CH3: CONN_2, symbol CONN_2
- removed CON3_VF_MOD, CON5, KEY: CONN_5, symbol CONN_5
- removed CON4_ISP: CONN_6, symbol CONN_6
- removed D1, D2, D3: DIODE, symbol DIODE
- removed LCD1: CONN_8, symbol CONN_8
- removed Q? (x4): KSC1623, symbol NPN
- removed SW1: DUAL_SWITCH_INV, symbol DUAL_SWITCH_INV
- removed U1: MIC5205-5.0BM5, symbol LT1761
- removed X1: CRYSTAL, symbol CRYSTAL
- added 3k9 (x2): R, symbol R
- added C?: C, symbol C
- added D1, D2, D3: D, symbol D
- added IC?: 24LC128, SO8, symbol AT24CS64-SSHM
- added P_ALT (x2), P_CH2, P_D/R: CONN_01X03, symbol CONN_01X03
- added P_ANT: CONN_01X01, symbol CONN_01X01
- added P_BATT, P_CH3: CONN_01X02, symbol CONN_01X02
- added P_ISP: CONN_01X06, symbol CONN_01X06
- added P_KEY, P_RF_MOD, P_TRIM: CONN_01X05, symbol CONN_01X05
- added P_LCD: CONN_01X08, symbol CONN_01X08
- added Q? (x4): KSC1623, symbol Q_NPN_EBC
- added SW1: Switch_SPDT_x2, symbol Switch_SPDT_x2
- added U?: MIC5205-5.0BM5, symbol LT1761-5
- added Y?: Crystal, symbol Crystal
Connections:
- net labels added: SCL, SDA
- wire segments 229 -> 249
- no-connect marks 7 -> 8
Other:
- note added: "(MOD)"
- note added: "External EEPROM"
- note added: "constantly connected to battery"
- note added: "for lower analog in crosstalk decrease\n(short) or 120R is ok"
- note removed: "for lower interference decrease\n(short) 120R is ok"
- moved on the sheet: C10, C11, C12, C13, C18, C19, C20, C21, C22, C23, C24, C25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
